Commit message: Add info about about ros2_control issue

File: panther_description/urdf/body.urdf.xacro (robot description, xacro)
@@ -4,14 +4,20 @@
   <xacro:macro
     name="body"
-    params="wheel_radius
+    params="namespace wheel_radius
             imu_pos_x imu_pos_y imu_pos_z
             imu_rot_r imu_rot_p imu_rot_y">
-    <link name="base_link" />
+    <xacro:if value="${namespace == ''}">
+      <xacro:property name="ns" value="" />
+    </xacro:if>
+    <xacro:unless value="${namespace == ''}">
+        <xacro:property name="ns" value="${namespace}/" />
+    </xacro:unless>
+    <link name="${ns}base_link" />
     <joint name="base_to_body_joint" type="fixed">
       <origin xyz="0.0 0.0 ${wheel_radius}" rpy="0.0 0.0 0.0" />
-      <parent link="base_link" />
-      <child link="body_link" />
+      <parent link="${ns}base_link" />
+      <child link="${ns}body_link" />
     </joint>
-    <link name="body_link">
+    <link name="${ns}body_link">
       <visual>
         <origin xyz="0.0 0.0 0.0" rpy="0.0 0.0 0.0" />
@@ -37,38 +43,38 @@
       <origin xyz="${imu_pos_x} ${imu_pos_y} ${imu_pos_z}"
         rpy="${imu_rot_r} ${imu_rot_p} ${imu_rot_y}" />
-      <parent link="body_link" />
-      <child link="imu_link" />
+      <parent link="${ns}body_link" />
+      <child link="${ns}imu_link" />
     </joint>
-    <link name="imu_link" />
+    <link name="${ns}imu_link" />
     <joint name="body_to_front_bumper_joint" type="fixed">
       <origin xyz="0.362 0.0 0.0" rpy="0.0 0.0 0.0" />
-      <parent link="body_link" />
-      <child link="front_bumper_link" />
+      <parent link="${ns}body_link" />
+      <child link="${ns}front_bumper_link" />
     </joint>
-    <link name="front_bumper_link" />
+    <link name="${ns}front_bumper_link" />
     <joint name="front_bumper_to_front_light_joint" type="fixed">
       <origin xyz="0.0 0.0 0.0185" rpy="${pi/2} 0.0 ${pi/2}" />
-      <parent link="front_bumper_link" />
-      <child link="front_light_link" />
+      <parent link="${ns}front_bumper_link" />
+      <child link="${ns}front_light_link" />
     </joint>
-    <link name="front_light_link" />
+    <link name="${ns}front_light_link" />
     <joint name="body_to_rear_bumper_joint" type="fixed">
       <origin xyz="-0.362 0.0 0.0" rpy="0.0 0.0 ${pi}" />
-      <parent link="body_link" />
-      <child link="rear_bumper_link" />
+      <parent link="${ns}body_link" />
+      <child link="${ns}rear_bumper_link" />
     </joint>
-    <link name="rear_bumper_link" />
+    <link name="${ns}rear_bumper_link" />
     <joint name="rear_bumper_to_rear_light_joint" type="fixed">
       <origin xyz="0.0 0.0 0.0185" rpy="${pi/2} 0.0 ${pi/2}" />
-      <parent link="rear_bumper_link" />
-      <child link="rear_light_link" />
+      <parent link="${ns}rear_bumper_link" />
+      <child link="${ns}rear_light_link" />
     </joint>
-    <link name="rear_light_link" />
+    <link name="${ns}rear_light_link" />
     <joint name="body_to_cover_joint" type="fixed">
       <origin xyz="0.0 0.0 0.1715" rpy="0.0 0.0 0.0" />
-      <parent link="body_link" />
-      <child link="cover_link" />
+      <parent link="${ns}body_link" />
+      <child link="${ns}cover_link" />
     </joint>
-    <link name="cover_link" />
+    <link name="${ns}cover_link" />
   </xacro:macro>
 </robot>

File: panther_description/urdf/panther_macro.urdf.xacro (robot description, xacro)
@@ -30,4 +30,5 @@
     <!-- BODY DECLARATION -->
     <xacro:body.body
+      namespace="${namespace}"
       wheel_radius="${wheel_config['wheel_radius']}"
       imu_pos_x="${imu_pos_x}"
@@ -39,16 +40,20 @@
     <!-- WHEEL DECLARATION -->
     <xacro:wheel.wheel
+      namespace="${namespace}"
       wheel_config="${wheel_config}"
       wheel_separation_x="${wheel_separation_x}"
       prefix="fl" />
     <xacro:wheel.wheel
+      namespace="${namespace}"
       wheel_config="${wheel_config}"
       wheel_separation_x="${wheel_separation_x}"
       prefix="fr" />
     <xacro:wheel.wheel
+      namespace="${namespace}"
       wheel_config="${wheel_config}"
       wheel_separation_x="${wheel_separation_x}"
       prefix="rl" />
     <xacro:wheel.wheel
+      namespace="${namespace}"
       wheel_config="${wheel_config}"
       wheel_separation_x="${wheel_separation_x}"
@@ -166,5 +171,5 @@
       <xacro:gazebo.battery config_file="${battery_config_file}" namespace="${namespace}" />
       <xacro:gazebo.controller config_file="${controller_config_file}" namespace="${namespace}" />
-      <xacro:gazebo.imu reference_frame="imu_link" namespace="${namespace}" />
+      <xacro:gazebo.imu reference_frame="${ns}imu_link" namespace="${namespace}" />
     </xacro:if>
   </xacro:macro>

File: panther_description/urdf/wheel.urdf.xacro (robot description, xacro)
@@ -2,5 +2,11 @@
 <robot xmlns:xacro="http://wiki.ros.org/xacro">
   <!-- wheel defining macro -->
-  <xacro:macro name="wheel" params="wheel_config wheel_separation_x prefix">
+  <xacro:macro name="wheel" params="namespace wheel_config wheel_separation_x prefix">
+  <xacro:if value="${namespace == ''}">
+    <xacro:property name="ns" value="" />
+  </xacro:if>
+  <xacro:unless value="${namespace == ''}">
+      <xacro:property name="ns" value="${namespace}/" />
+  </xacro:unless>
     <xacro:if value="${prefix == 'fl'}">
       <xacro:property name="x" value="${wheel_separation_x/2.0}" />
@@ -29,11 +35,11 @@
     <joint name="${prefix}_wheel_joint" type="continuous">
       <origin xyz="${x} ${y} 0.0" rpy="0.0 0.0 0.0" />
-      <parent link="body_link" />
-      <child link="${prefix}_wheel_link" />
+      <parent link="${ns}body_link" />
+      <child link="${ns}${prefix}_wheel_link" />
       <axis xyz="0.0 1.0 0.0" />
       <limit effort="64.5" velocity="10.958" />
       <dynamics damping="0.01" friction="0.1" />
     </joint>
-    <link name="${prefix}_wheel_link">
+    <link name="${ns}${prefix}_wheel_link">
       <visual>
         <origin xyz="0.0 0.0 0.0" rpy="0.0 0.0 0.0" />
@@ -62,5 +68,5 @@
     </link>
     <xacro:if value="${use_sim}">
-      <gazebo reference="${prefix}_wheel_link" xmlns:ignition="http://ignitionrobotics.org/schema">
+      <gazebo reference="${ns}${prefix}_wheel_link" xmlns:ignition="http://ignitionrobotics.org/schema">
         <collision>
           <surface>
@@ -69,5 +75,5 @@
                 <mu>1.0</mu>
                 <mu2>0.0</mu2>
-                <fdir1 ignition:expressed_in="base_link">${fdir}</fdir1>
+                <fdir1 ignition:expressed_in="${ns}base_link">${fdir}</fdir1>
               </ode>
             </friction>
